File: astrodewar-mas-4L-flex-vertical-mount.kicad_pcb (KiCad board)
At the start: 4 copper layers, 288.3 x 67.3 mm, 2 parts, among them J1 Conn_02x25_Top_Bottom, U1 DB-50-LTA-V2

Commit message: Reduced length of tapering
To accommodate astro dewar restrictions at the feedthrough.
Other:
- board size 288.3 x 67.3 mm -> 280.3 x 67.3 mm
- board text added: "MAS Flex (4 layers) April 2024 Kenneth Lin Alex Drlica-Wagner Claudio Chavez"
- board text added: "Serial No."
- board text added: "Stiffener (TOP)"

Commit message: Clock jumps layer change
And added silkscreen.
Parts:
- added G***: LOGO, projectFootprints:fnal_logo, F.Cu at (333.4, 136.5)
- added G***: LOGO, projectFootprints:cal, F.Cu at (320.5, 136.7)
Other:
- outline, holes or cut-outs redrawn
- board text added: "MAS Flex (4 layers)"
